File: ble_bme690_node.brd (EAGLE design)
At the start: 47 x 47 mm, 56 parts, among them IC1 ZMOD4510AI1R, J1 JTAG, J2 TYPE-C-31-M-12, U1 ESP32-C6-MINI-1-N4, U2 BME690, U3 TPS63001DRCR, U4 LM66100DCKR, U5 LM66100DCKR, U6 XTSD04GLGEAG, Y1 Q13FC13500003

Commit message: Completed design files
Parts:
- removed J6: (no value), SparkFun-Connectors:JST-2-SMD
- removed R3: 10M, SparkFun-Resistors:0603
- added C22, C24: 0.1uF, SparkFun-Capacitors:0402
- added C23, C25: 0.1uF, SparkFun-Capacitors_Sai:0402
- added J3: SM06B-GHS-TB(LF)(SN), SM06B-GHS-TB_LF__SN_:JST_SM06B-GHS-TB(LF)(SN)
- added J4: S2B-PH-K-S, SparkFun-Connectors:JST-2-PTH-NS
- added LED1: WS2812B-2020, WS2812B-2020:WS2812B-2020
- added U7: PCF8563T/F4,118, PCF8563T_F4_118:SOIC127P600X175-8N
- C10, C14, C15, C16, C17, C18, C2, C20, C21, C4, C5, C6, C9: device SparkFun-Capacitors:0603 -> SparkFun-Capacitors_Sai:0402
- C11, C12, C13: value 10uF -> 10UF0402; device SparkFun-Capacitors:0603 -> SparkFun-Capacitors_Sai:0402
- C19: value 4.7uF -> 4.7UF0402; device SparkFun-Capacitors:0603 -> SparkFun-Capacitors_Sai:0402
- J5: value (none) -> SM04B-SRSS-TB(LF)(SN)
- R1, R15, R2, R4, R5, R6, R7, R8: device SparkFun-Resistors:0603 -> SparkFun-Resistors_Sai:0402
- R10, R13: value 100 -> 100OHM; device SparkFun-Resistors:0603 -> SparkFun-Resistors_Sai:0402
- R14: value 2.0k -> 2.0K; device SparkFun-Resistors:0603 -> SparkFun-Resistors_Sai:0402
- moved U6 86.3 mm to (36.3, 36.2), turned to 180 degrees
- moved R12 84.9 mm to (38.6, 15.3), turned to 180 degrees
- moved R11 83.0 mm to (38.6, 16.7), turned to 180 degrees
- moved R9 68.7 mm to (31.5, 7.95), turned to 180 degrees
- moved C21 63.5 mm to (38.8, 8.31), turned to 270 degrees
- moved C20 56.1 mm to (31.5, 9.35)
- moved C17 54.1 mm to (31.2, 14.2)
- moved C18 52.0 mm to (31.5, 6.53)
- moved C15 50.8 mm to (31.2, 12.4)
- moved U2 46.0 mm to (34.4, 12.9)
- moved IC1 45.5 mm to (35.5, 7.62)
- moved R14 13.7 mm to (9.30, 18.3), turned to 90 degrees
- moved R13 10.3 mm to (43.3, 34.1), turned to 180 degrees
- moved C6 8.50 mm to (12.3, 17.9), turned to 180 degrees
- moved U$1 7.84 mm to (8.33, 22.7), turned to 270 degrees
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Connections:
- removed net RTC_OUT: C5.1, R3.1, U1.12, Y1.2
- removed net VDD: U6.8
- removed net VSS: U6.4
- new net !CS: U1.20, U6.2
- new net !INT_RTC: U1.13, U7.3
- new net MISO: U1.25, U6.6
- new net MOSI: U1.26, U6.5
- new net N$8: C5.1, U7.1, Y1.2
- new net NEOPIXEL: LED1.3, U1.19
- new net SCK: U1.24, U6.3
- net !RST_ZMOD4510: now also U1.28
- net 3.3V: now also C23.2, C24.1, C25.1, LED1.4, U6.8, U7.8
- net GND: now also C22.2, C23.1, C24.2, C25.2, J3.2, J3.5, J3.S1, J3.S2, J4.1, LED1.2, U6.4, U7.4; no longer J6.1
- net INT_ZMOD4510: now also U1.27
- net RTC_IN: now also U7.2; no longer R3.2, U1.13
- net SCL: now also J3.4, U7.6
- net SDA: now also J3.3, U7.5
- net V_BATT: now also J4.2; no longer J6.2
- net V_USB_2: now also C22.1, J3.1
Routing:
- net SCL: track 51.2 -> 110.5 mm, vias 4 -> 6
- net INT_ZMOD4510: track 0.00 -> 38.3 mm, vias 0 -> 2
- net V_USB_2: track 34.1 -> 72.0 mm, vias 3 -> 4
- net !RST_ZMOD4510: track 0.00 -> 36.0 mm, vias 0 -> 2
- net SDA: track 60.6 -> 94.5 mm, vias 2 -> 5
- net 3.3V: track 27.5 -> 51.4 mm, vias 7 -> 16
- net SCK: track 0.00 -> 20.9 mm
- net !CS: track 0.00 -> 20.6 mm, vias 0 -> 2
- net N$11: track 3.49 -> 19.0 mm, vias 0 -> 2
- net !INT_RTC: track 0.00 -> 14.3 mm
- net NEOPIXEL: track 0.00 -> 11.5 mm, vias 0 -> 2
- net MOSI: track 0.00 -> 9.43 mm
- net N$15: track 10.9 -> 1.50 mm, vias 2 -> 0
- net MISO: track 0.00 -> 8.91 mm
- net V_BATT: track 25.2 -> 17.6 mm
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Other:
- board text added: "PM Sensor"
- board text added: "Qwiic"
