File: ble_bme690_node.sch (EAGLE design)
At the start: 56 parts, among them IC1 ZMOD4510AI1R, J1 JTAG, J2 TYPE-C-31-M-12, U1 ESP32-C6-MINI-1-N4, U2 BME690, U3 TPS63001DRCR, U4 LM66100DCKR, U5 LM66100DCKR, U6 XTSD04GLGEAG, Y1 Q13FC13500003

Commit message: Completed design files
Parts:
- removed J6: (no value), SparkFun-Connectors:JST_2MM_MALE
- removed R3: 10M, SparkFun-Resistors:10MOHM-0603-1/10W-5%
- added C22, C24: 0.1uF, SparkFun-Capacitors:0.1UF-0402-16V-10%
- added C23, C25: 0.1uF, SparkFun-Capacitors_Sai:0.1UF-0402-6.3V-10%-X7R
- added J3: SM06B-GHS-TB(LF)(SN), SM06B-GHS-TB_LF__SN_:SM06B-GHS-TB(LF)(SN)
- added J4: S2B-PH-K-S, SparkFun-Connectors:CONN_02-JST-2-PTH-NO_SILK
- added LED1: WS2812B-2020, WS2812B-2020:WS2812B-2020
- added U7: PCF8563T/F4,118, PCF8563T_F4_118:PCF8563T/F4,118
- C10, C14, C15, C16, C17, C18, C2, C20, C21, C4, C9: device SparkFun-Capacitors:0.1UF-0603-25V-(+80/-20%) -> SparkFun-Capacitors_Sai:0.1UF-0402-6.3V-10%-X7R
- C11, C12, C13: value 10uF -> 10UF0402; device SparkFun-Capacitors:10UF-0603-6.3V-20% -> SparkFun-Capacitors_Sai:10UF0402
- C19: value 4.7uF -> 4.7UF0402; device SparkFun-Capacitors:4.7UF-0603-6.3V-(10%) -> SparkFun-Capacitors_Sai:4.7UF0402
- C5, C6: device SparkFun-Capacitors:12PF-0603-50V-5% -> SparkFun-Capacitors_Sai:12PF-0402-50V-5%
- J5: value (none) -> SM04B-SRSS-TB(LF)(SN)
- R1, R6: device SparkFun-Resistors:10KOHM-0603-1/10W-1% -> SparkFun-Resistors_Sai:10KOHM-0402-1/16W-1%
- R10, R13: value 100 -> 100OHM; device SparkFun-Resistors:100OHM-0603-1/10W-1% -> SparkFun-Resistors_Sai:100OHM
- R14: value 2.0k -> 2.0K; device SparkFun-Resistors:2.0KOHM-0603-1/10W-5% -> SparkFun-Resistors_Sai:2.0KOHM-0402-1/16W-1%
- R15: device SparkFun-Resistors:470OHM-0603-1/10W-1% -> SparkFun-Resistors_Sai:470OHM-0402-1/16W-5%
- R2, R4, R5: device SparkFun-Resistors:0OHM-0603-1/10W -> SparkFun-Resistors_Sai:0OHM-0402-1/10W
- R7, R8: device SparkFun-Resistors:5.1KOHM5.1KOHM-0603-1/10W-1% -> SparkFun-Resistors_Sai:5.1KOHM-0402-1/16W-1%
Connections:
- removed net RTC_OUT: C5.1, R3.1, U1.IO0, Y1.2
- new net !CS: U1.IO15, U6.SD3/!CS
- new net !INT_RTC: U1.IO1, U7.~INT
- new net MISO: U1.IO19, U6.SD0/DO
- new net MOSI: U1.IO20, U6.CMD/DI
- new net N$8: C5.1, U7.OSCI, Y1.2
- new net NEOPIXEL: LED1.DI, U1.IO14
- new net SCK: U1.IO18, U6.CLK
- net !RST_ZMOD4510: now also U1.IO22
- net 3.3V: now also C23.2, C24.1, C25.1, LED1.VDD, U6.VDD, U7.VDD
- net GND: now also C22.2, C23.1, C24.2, C25.2, J3.2, J3.5, J3.SHIELD, J4.1, LED1.VSS, U6.VSS, U7.VSS; no longer J6.-
- net INT_ZMOD4510: now also U1.IO21
- net RTC_IN: now also U7.OSCO; no longer R3.2, U1.IO1
- net SCL: now also J3.4, U7.SCL
- net SDA: now also J3.3, U7.SDA
- net V_BATT: now also J4.2; no longer J6.+
- net V_USB_2: now also C22.1, J3.1
Other:
- note added: "Address: 0x69"
- note added: "Dust Sensor"
- moved on the sheet: C5, C6, Y1
