File: ble_bme690_node_1.kicad_sch (KiCad schematic)
At the start: 40 parts, among them IC1 ZMOD4510AI1R, J1 JTAG, J3 SM06B-GHS-TB(LF)(SN), J5 SM04B-SRSS-TB(LF)(SN), U1 ESP32-C6-MINI-1-N4, U2 BME690, U6 XTSD04GLGEAG, U7 PCF8563T/F4,118, Y1 Q13FC13500003

Commit message: code checked in
Parts:
- removed BOOT0, RESET0: MOMENTARY-SWITCH-SPST-SMD-4.6X2.8MM, KiCAD_converted:TACTILE_SWITCH_SMD_4.6X2.8MM, symbol KiCAD_converted-eagle-import:MOMENTARY-SWITCH-SPST-SMD-4.6X2.8MM
- removed C1: 22uF, KiCAD_converted:0603, symbol KiCAD_converted-eagle-import:22UF-0603-6.3V-20%
- removed C22, C24: 0.1uF, KiCAD_converted:0402, symbol KiCAD_converted-eagle-import:0.1UF-0402-16V-10%
- removed C3: 1.0uF, KiCAD_converted:0402, symbol KiCAD_converted-eagle-import:1.0UF-0402-16V-10%
- removed C5, C6: 12pF, KiCAD_converted:0402, symbol KiCAD_converted-eagle-import:12PF-0402-50V-5%
- removed C7, C8: DNP, KiCAD_converted:0402, symbol KiCAD_converted-eagle-import:0.1UF-0402-6.3V-10%-X7R
- removed D2: RED, KiCAD_converted:LED-0603, symbol KiCAD_converted-eagle-import:LED-RED0603
- removed IC1: ZMOD4510AI1R, KiCAD_converted:ZMOD4510AI1R, symbol KiCAD_converted-eagle-import:ZMOD4510AI1R
- removed J1: JTAG, KiCAD_converted:2X5-SMD-UNSHROUDED, symbol KiCAD_converted-eagle-import:CORTEX_JTAG_DEBUG_SMD-UNSHROUDED
- removed J3: SM06B-GHS-TB(LF)(SN), KiCAD_converted:JST_SM06B-GHS-TB(LF)(SN), symbol KiCAD_converted-eagle-import:SM06B-GHS-TB(LF)(SN)
- removed J5: SM04B-SRSS-TB(LF)(SN), KiCAD_converted:1X04_1MM_RA, symbol KiCAD_converted-eagle-import:QWIIC_CONNECTORJS-1MM
- removed LED1: WS2812B-2020, KiCAD_converted:WS2812B-2020, symbol KiCAD_converted-eagle-import:WS2812B-2020
- removed R1, R11, R12, R6, R9: 10k, KiCAD_converted:0402, symbol KiCAD_converted-eagle-import:10KOHM-0402-1/16W-1%
- removed R13: 100OHM, KiCAD_converted:0402, symbol KiCAD_converted-eagle-import:100OHM
- removed R2, R4, R5: 0, KiCAD_converted:0402, symbol KiCAD_converted-eagle-import:0OHM-0402-1/10W
- removed U1: ESP32-C6-MINI-1-N4, KiCAD_converted:XCVR_ESP32-C6-MINI-1-N4, symbol KiCAD_converted-eagle-import:ESP32-C6-MINI-1-N4
- removed U2: BME690, KiCAD_converted:IC_BME688, symbol KiCAD_converted-eagle-import:BME690
- removed U6: XTSD04GLGEAG, KiCAD_converted:SON127P600X800X95-8N, symbol KiCAD_converted-eagle-import:XTSD04GLGEAG
- removed U7: PCF8563T/F4,118, KiCAD_converted:SOIC127P600X175-8N, symbol KiCAD_converted-eagle-import:PCF8563T/F4,118
- removed Y1: Q13FC13500003, KiCAD_converted:XTAL_FC-135_32.7680KA-A0, symbol KiCAD_converted-eagle-import:FC-135_32.7680KA-A0
- added BOOT0, RESET0: MOMENTARY-SWITCH-SPST-SMD-4.6X2.8MM, KiCAD_converted:TACTILE_SWITCH_SMD_4.6X2.8MM, symbol KiCAD_converted-eagle-import:SparkFun-Switches_535_MOMENTARY-SWITCH-SPST-SMD-4.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
- added C1: 22uF, KiCAD_converted:0603, symbol KiCAD_converted-eagle-import:SparkFun-Capacitors_510_22UF-0603-6.3V-20%
- added C22, C24: 0.1uF, KiCAD_converted:0402, symbol KiCAD_converted-eagle-import:SparkFun-Capacitors_510_0.1UF-0402-16V-10%
- added C3: 1.0uF, KiCAD_converted:0402, symbol KiCAD_converted-eagle-import:SparkFun-Capacitors_Sai_1.0UF-0402-16V-10%
- added C5, C6: 12pF, KiCAD_converted:0402, symbol KiCAD_converted-eagle-import:SparkFun-Capacitors_Sai_12PF-0402-50V-5%
- added C7, C8: DNP, KiCAD_converted:0402, symbol KiCAD_converted-eagle-import:SparkFun-Capacitors_510_0.1UF-0402-6.3V-10%-X7R
- added D2: RED, KiCAD_converted:LED-0603, symbol KiCAD_converted-eagle-import:SparkFun-LED_529_LED-RED0603
- added IC1: ZMOD4510AI1R, KiCAD_converted:ZMOD4510AI1R, symbol KiCAD_converted-eagle-import:ZMOD4510AI1R_ZMOD4510AI1R
- added J1: JTAG, KiCAD_converted:2X5-SMD-UNSHROUDED, symbol KiCAD_converted-eagle-import:SparkFun-Connectors_513_CORTEX_JTAG_DEBUG_SMD-UNSH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
- added J3: SM06B-GHS-TB(LF)(SN), KiCAD_converted:JST_SM06B-GHS-TB(LF)(SN), symbol KiCAD_converted-eagle-import:SM06B-GHS-TB_LF__SN__SM06B-GHS-TB(LF)(SN)
- added J5: SM04B-SRSS-TB(LF)(SN), KiCAD_converted:1X04_1MM_RA, symbol KiCAD_converted-eagle-import:SparkFun-Connectors_2652347_QWIIC_CONNECTORJS-1MM
- added LED1: WS2812B-2020, KiCAD_converted:WS2812B-2020, symbol KiCAD_converted-eagle-import:WS2812B-2020_WS2812B-2020
- added R1, R11, R12, R6, R9: 10k, KiCAD_converted:0402, symbol KiCAD_converted-eagle-import:SparkFun-Resistors_Sai_10KOHM-0402-1/16W-1%
- added R13: 100OHM, KiCAD_converted:0402, symbol KiCAD_converted-eagle-import:SparkFun-Resistors_Sai_100OHM
- added R2, R4, R5: 0, KiCAD_converted:0402, symbol KiCAD_converted-eagle-import:SparkFun-Resistors_Sai_0OHM-0402-1/10W
- added U1: ESP32-C6-MINI-1-N4, KiCAD_converted:XCVR_ESP32-C6-MINI-1-N4, symbol KiCAD_converted-eagle-import:ESP32-C6-MINI-1-N4_ESP32-C6-MINI-1-N4
- added U2: BME690, KiCAD_converted:IC_BME688, symbol KiCAD_converted-eagle-import:BME690_BME690
- added U6: XTSD04GLGEAG, KiCAD_converted:SON127P600X800X95-8N, symbol KiCAD_converted-eagle-import:XTSD04GLGEAG_XTSD04GLGEAG
- added U7: PCF8563T/F4,118, KiCAD_converted:SOIC127P600X175-8N, symbol KiCAD_converted-eagle-import:PCF8563T_F4_118_PCF8563T/F4,118
- added Y1: Q13FC13500003, KiCAD_converted:XTAL_FC-135_32.7680KA-A0, symbol KiCAD_converted-eagle-import:FC-135_32.7680KA-A0_FC-135_32.7680KA-A0
Connections:
- net 3.3V: now also C1.1, C24.1, IC1.10 (VDDH), IC1.12 (VDDIO), IC1.5 (VDD), J1.1 (VCC), J5.2, LED1.4 (VDD), R1.2, R11.2, R12.2, R6.2, R9.2, U1.3 (3V3), U2.2 (CSB), U2.6 (VDDIO), U2.8 (VDD), U6.8 (VDD), U7.8 (VDD)
- net EN: now also C3.2, J1.10 (~{RESET}), R1.1, R2.2, U1.8 (EN)
- net GND: now also BOOT0.1, BOOT0.2 (1), C1.2, C22.2, C24.2, C3.1, C5.2, C6.2, C7.2, C8.2, D2.C, IC1.6 (VSS_1), IC1.7 (VSS_2), IC1.9 (VSS_3), J1.3 (GND@3), J1.5 (GND@5), J1.9 (GNDDTCT), J3.2, J3.5, J3.S1 (SHIELD), J3.S2 (SHIELD), J5.1, LED1.2 (VSS), RESET0.1, RESET0.2 (1), U1.1 (GND1), U1.11 (GND1), U1.14 (GND1), U1.2 (GND1), U1.36 (GND1), U1.37 (GND1), U1.38 (GND1), U1.39 (GND1), U1.40 (GND1), U1.41 (GND1), U1.42 (GND1), U1.43 (GND1), U1.44 (GND1), U1.45 (GND1), U1.46 (GND1), U1.47 (GND2), U1.48 (GND2), U1.49_1 (GND2), U1.49_2 (GND2), U1.49_3 (GND2), U1.49_4 (GND2), U1.49_5 (GND2), U1.49_6 (GND2), U1.49_7 (GND2), U1.49_8 (GND2), U1.49_9 (GND2), U1.50 (GND2), U1.51 (GND2), U1.52 (GND2), U1.53 (GND2), U2.1 (GND), U2.5 (SDO), U2.7 (GND), U6.4 (VSS), U7.4 (VSS)
- net INT_ZMOD4510: now also IC1.3 (INT), U1.27 (IO21)
- net MISO: now also U1.25 (IO19), U6.6 (SD0/DO)
- net MOSI: now also U1.26 (IO20), U6.5 (CMD/DI)
- net NEOPIXEL: now also LED1.3 (DI), U1.19 (IO14)
- net SCK: now also U1.24 (IO18), U6.3 (CLK)
- net SCL: now also IC1.1 (SCL), J3.4, J5.4, R11.1, U1.5 (IO2), U2.4 (SCK), U7.6 (SCL)
- net SDA: now also IC1.2 (SDA), J3.3, J5.3, R12.1, U1.6 (IO3), U2.3 (SDI), U7.5 (SDA)
- net TCK: now also J1.4 (SWDCLK/TCK), U1.15 (IO6)
- net TDI: now also J1.8 (NC/TDI), U1.10 (IO5)
- net TDO: now also J1.6 (SWO/TDO), U1.16 (IO7)
- net TMS: now also J1.2 (SWDIO/TMS), U1.9 (IO4)
- net USB_N: now also C8.1, R5.2
- net USB_P: now also C7.1, R4.2
- net V_USB_IN: now also C22.1, J3.1
- net ~{BOOT}: now also BOOT0.3 (2), BOOT0.4 (2), U1.23 (IO9)
- net ~{CS}: now also U1.20 (IO15), U6.2 (SD3/~{CS})
- net ~{INT_RTC}: now also U1.13 (IO1), U7.3 (~{INT})
- net ~{RESET}: now also R2.1, RESET0.3 (2), RESET0.4 (2)
- net ~{RST_ZMOD4510}: now also IC1.11 (RES_N), R9.1, U1.28 (IO22)
- new net: R6.1, U1.22 (IO8)
- new net: R5.1, U1.17 (IO12)
- new net: C6.1, U7.2 (OSCO), Y1.1
- new net: C5.1, U7.1 (OSCI), Y1.2
- new net: R13.1, U1.29 (IO23)
- new net: D2.A, R13.2
- new net: R4.1, U1.18 (IO13)
- new net: U1.21 (NC), U1.32 (NC), U1.33 (NC), U1.34 (NC), U1.35 (NC), U1.4 (NC), U1.7 (NC)
