File: ble_bme690_node_2.kicad_sch (KiCad schematic)
At the start: 22 parts, among them J2 TYPE-C-31-M-12, J4 S2B-PH-K-S, U3 TPS63001DRCR, U4 LM66100DCKR, U5 LM66100DCKR

Commit message: code checked in
Parts:
- removed C11, C12, C13: 10UF0402, KiCAD_converted:0402, symbol KiCAD_converted-eagle-import:10UF0402
- removed C19: 4.7UF0402, KiCAD_converted:0402, symbol KiCAD_converted-eagle-import:4.7UF0402
- removed D3: RED, KiCAD_converted:LED-0603, symbol KiCAD_converted-eagle-import:LED-RED0603
- removed J2: TYPE-C-31-M-12, KiCAD_converted:HRO_TYPE-C-31-M-12, symbol KiCAD_converted-eagle-import:TYPE-C-31-M-12
- removed J4: S2B-PH-K-S, KiCAD_converted:JST-2-PTH-NS, symbol KiCAD_converted-eagle-import:CONN_02-JST-2-PTH-NO_SILK
- removed L1: 2.2nH, KiCAD_converted:0603, symbol KiCAD_converted-eagle-import:3.9NH
- removed L2: NR3015T2R2M, KiCAD_converted:IND_NR3015T2R2M, symbol KiCAD_converted-eagle-import:NR3015T2R2M
- removed R10: 100OHM, KiCAD_converted:0402, symbol KiCAD_converted-eagle-import:100OHM
- removed R14: 2.0K, KiCAD_converted:0402, symbol KiCAD_converted-eagle-import:2.0KOHM-0402-1/16W-1%
- removed R15: 470, KiCAD_converted:0402, symbol KiCAD_converted-eagle-import:470OHM-0402-1/16W-5%
- removed R7, R8: 5.1k, KiCAD_converted:0402, symbol KiCAD_converted-eagle-import:5.1KOHM-0402-1/16W-1%
- removed S1: JS202011JCQN, KiCAD_converted:SW_JS202011JCQN, symbol KiCAD_converted-eagle-import:JS202011JCQN
- removed U$1: MCP73831T-2ACI/OT, KiCAD_converted:SOT95P280X145-5N, symbol KiCAD_converted-eagle-import:MCP73831T-2ACI/OT
- removed U3: TPS63001DRCR, KiCAD_converted:VREG_V62_16624-01YE, symbol KiCAD_converted-eagle-import:TPS63001DRCR
- removed U4, U5: LM66100DCKR, KiCAD_converted:SOT65P210X110-6N, symbol KiCAD_converted-eagle-import:LM66100DCKR
- added C11, C12, C13: 10UF0402, KiCAD_converted:0402, symbol KiCAD_converted-eagle-import:SparkFun-Capacitors_Sai_10UF0402
- added C19: 4.7UF0402, KiCAD_converted:0402, symbol KiCAD_converted-eagle-import:SparkFun-Capacitors_Sai_4.7UF0402
- added D3: RED, KiCAD_converted:LED-0603, symbol KiCAD_converted-eagle-import:SparkFun-LED_529_LED-RED0603
- added J2: TYPE-C-31-M-12, KiCAD_converted:HRO_TYPE-C-31-M-12, symbol KiCAD_converted-eagle-import:TYPE-C-31-M-12_TYPE-C-31-M-12
- added J4: S2B-PH-K-S, KiCAD_converted:JST-2-PTH-NS, symbol KiCAD_converted-eagle-import:SparkFun-Connectors_2652347_CONN_02-JST-2-PTH-NO_S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
- added L1: 2.2nH, KiCAD_converted:0603, symbol KiCAD_converted-eagle-import:SparkFun-Coils_512_3.9NH
- added L2: NR3015T2R2M, KiCAD_converted:IND_NR3015T2R2M, symbol KiCAD_converted-eagle-import:NR3015T2R2M_NR3015T2R2M
- added R10: 100OHM, KiCAD_converted:0402, symbol KiCAD_converted-eagle-import:SparkFun-Resistors_Sai_100OHM
- added R14: 2.0K, KiCAD_converted:0402, symbol KiCAD_converted-eagle-import:SparkFun-Resistors_Sai_2.0KOHM-0402-1/16W-1%
- added R15: 470, KiCAD_converted:0402, symbol KiCAD_converted-eagle-import:SparkFun-Resistors_Sai_470OHM-0402-1/16W-5%
- added R7, R8: 5.1k, KiCAD_converted:0402, symbol KiCAD_converted-eagle-import:SparkFun-Resistors_Sai_5.1KOHM-0402-1/16W-1%
- added S1: JS202011JCQN, KiCAD_converted:SW_JS202011JCQN, symbol KiCAD_converted-eagle-import:JS202011JCQN_JS202011JCQN
- added U$1: MCP73831T-2ACI/OT, KiCAD_converted:SOT95P280X145-5N, symbol KiCAD_converted-eagle-import:MCP73831T-2ACI_OT_MCP73831T-2ACI/OT
- added U3: TPS63001DRCR, KiCAD_converted:VREG_V62_16624-01YE, symbol KiCAD_converted-eagle-import:TPS63001DRCR_TPS63001DRCR
- added U4, U5: LM66100DCKR, KiCAD_converted:SOT65P210X110-6N, symbol KiCAD_converted-eagle-import:LM66100DCKR_LM66100DCKR
Connections:
- net 3.3V: now also C11.1, C12.1, U3.1 (VOUT), U3.10 (FB)
- net GND: now also C11.2, C12.2, C13.1, C19.2, J2.A1_B12 (GND), J2.B1_A12 (GND), J2.S1 (SHIELD), J2.S2 (SHIELD), J2.S3 (SHIELD), J2.S4 (SHIELD), J4.1, R14.1, R15.1, R7.1, R8.1, U$1.2 (VSS), U3.11 (POWER_PAD), U3.12 (POWER_PAD), U3.13 (POWER_PAD), U3.14 (POWER_PAD), U3.15 (POWER_PAD), U3.3 (PGND), U3.9 (GND), U4.2 (GND), U5.2 (GND), U5.5 (ST)
- net USB_N: now also J2.A7 (DN1), J2.B7 (DN2)
- net USB_P: now also J2.A6 (DP1), J2.B6 (DP2)
- net VBUS_PREFILTER: now also J2.A4_B9 (VBUS), J2.B4_A9 (VBUS), L1.1
- net VIN: now also S1.3, U4.3 (~{CE}), U5.1 (VIN)
- net V_BATT: now also C19.1, J4.2, S1.2, U$1.3 (VBAT)
- net V_OR: now also C13.2, R10.1, U3.5 (VIN), U4.6 (VOUT), U5.6 (VOUT)
- net V_USB_IN: now also L1.2, U$1.4 (VDD), U4.1 (VIN), U5.3 (~{CE})
- net at C14.2: now also R10.2, U3.6 (EN), U3.7 (PS/SYNC), U3.8 (VINA)
- new net: D3.C, R15.2
- new net: J2.B5 (CC2), R7.2
- new net: L2.1, U3.2 (L2)
- new net: L2.2, U3.4 (L1)
- new net: J2.A5 (CC1), R8.2
- new net: D3.A, U$1.1 (STAT)
- new net: R14.2, U$1.5 (PROG)
