File: GHTC/RP2350/RP2350.kicad_sch (KiCad schematic)
At the start: 38 parts, among them IC1 W25Q64JVXGIQ, J1 SM03B-SRSS-TB_(LF)(SN), U1 RP2350A-QFN60, U2 APS6404L-3SQR-ZR, Y1 ABM8-272-T3

Commit message: Kicad schematic - daily backup.
Parts:
- removed IC1: W25Q64JVXGIQ, SamacSys_Parts:SON80P400X400X50-9N, symbol SamacSys_Parts:W25Q64JVXGIQ
- removed R8: 10K, SparkFun-Resistor:R_0402_1005Metric, symbol SparkFun-Resistor:1k_0402
- added C16, C21, C23, C26, C27: 0.1uF, SparkFun-Capacitor:C_0402_1005Metric, symbol SparkFun-Capacitor:0.1uF_0402_10V_10%
- added C24, C25: 10uF, Capacitor_SMD:C_0402_1005Metric, symbol SparkFun-Capacitor:10uF_0402_6.3V_20%
- added C28: 0.1uF, Capacitor_SMD:C_0402_1005Metric, symbol SparkFun-Capacitor:0.1uF_0402_10V_10%
- added C29, C30: 10uF, PCM_SparkFun-Capacitor:C_0402_1005Metric, symbol SparkFun-Capacitor:10uF_0402_6.3V_20%
- added IC1: STCC4-D-R3, SparkFun-Sensor:STCC4, symbol SamacSys_Parts:STCC4-D-R3
- added J2: 5035661302, 5035661302:CON_5035661302_MOL, symbol 5035661302:5035661302
- added J3: TYPE-C-31-M-12, TYPE-C-31-M-12:HRO_TYPE-C-31-M-12, symbol TYPE-C-31-M-12:TYPE-C-31-M-12
- added L2: 2.2nH, Inductor_SMD:L_0402_1005Metric, symbol SparkFun-Coil:2.2uH_0806_1.2A
- added R10, R8: 4.7k, Resistor_SMD:R_0402_1005Metric, symbol SparkFun-Resistor:4.7k_0402
- added R3, R4: 5.1k, PCM_SparkFun-Resistor:R_0402_1005Metric, symbol SparkFun-Resistor:5.1k_0402
- added U3: SHT4x, Sensor_Humidity:Sensirion_DFN-4_1.5x1.5mm_P0.8mm_SHT4x_NoCentralPad, symbol Sensor_Humidity:SHT4x
- added U4: BME688, BME688:IC_BME688, symbol BME688:BME688
- added U5: SGP41-D-R4, SGP41-D-R4:XDCR_SGP41-D-R4, symbol SGP41-D-R4:SGP41-D-R4
- added U6: ENS160-BGLM, ENS160-BGLM:XDCR_ENS160-BGLM, symbol ENS160-BGLM:ENS160-BGLM
- added U7: AZ1117CH2-3.3, Package_TO_SOT_SMD:SOT-223-3_TabPin2, symbol Regulator_Linear:AZ1117CH2-3.3
- U1: LCSC C42411118 -> C41378174
Connections:
- net ~{FLASH_SS} is gone; now on net ~{PSRAM_CS}: U1.2 (GPIO0)
- net +3.3V: now also C16.1, C21.1, C23.1, C24.2, C25.2, C26.1, C30.1, IC1.6 (VDDIO), IC1.7 (VDD), J2.1 (VDDL), J2.10 (VDDD), J2.3 (VDDA), J2.8 (VDDIO), R10.2, R8.2, U3.3 (VDD), U4.6 (VDDIO), U4.8 (VDD), U5.1 (VDD), U5.5 (VDDH), U6.4 (VDD), U6.5 (VDDIO), U7.3 (OUT)
- net GND: now also C16.2, C21.2, C23.2, C24.1, C25.1, C26.2, C27.2, C28.2, C29.2, C30.2, IC1.3 (ADDR), IC1.4 (VSS), J2.2 (VSSA), J2.7 (PS), J2.9 (VSSD), J3.A1_B12 (GND), J3.B1_A12 (GND__1), J3.S1 (SHIELD), J3.S2 (SHIELD__1), J3.S3 (SHIELD__2), J3.S4 (SHIELD__3), R3.1, R4.2, U3.4 (VSS), U4.1 (GND), U4.7 (GND__1), U5.2 (VSS), U5.7 (EXP), U6.8 (VSS), U6.9 (VSS__1), U7.2 (GND)
- net ~{PSRAM_CS}: no longer U1.12 (GPIO8)
- net ~{BMV080_CSB}: now reaches U1.13 (GPIO9)
- net ~{BMV080_CSB}: now also J2.4 (CSB)
- net ~{BME688_CSB}: now reaches U1.3 (GPIO1)
- net ~{BME688_CSB}: now also U4.2 (CSB)
- net I2C_SDA: now reaches U1.4 (GPIO2)
- net I2C_SDA: now also IC1.5 (SDA), R10.1, U5.3 (SDA)
- net I2C_SCL: now reaches U1.5 (GPIO3)
- net I2C_SCL: now also IC1.1 (SCL), R8.1, U5.6 (SCL)
- net MISO renamed SPI_MISO
- net SPI_MISO: now also J2.11 (MISO), U4.5 (SDO), U6.3 (MISO/ADDR)
- net MOSI renamed SPI_MOSI
- net SPI_MOSI: now also J2.5 (MOSI), U4.3 (SDI), U6.1 (MOSI/SDA)
- net SCK renamed SPI_SCK
- net SPI_SCK: now also J2.6 (SCK), U4.4 (SCK), U6.2 (SCLK/SCL)
- net USB+ renamed USBC.D+
- net USBC.D+: now also J3.A6 (DP1), J3.B6 (DP2)
- net USB- renamed USBC.D-
- net USBC.D-: now also J3.A7 (DN1), J3.B7 (DN2)
- net USB_N renamed USB_2354.D-
- net USB_P renamed USB_2354.D+
- net ~{CS_MEM} renamed ~{MEM_CS}
- net ~{INT_NPM1300} renamed BMV080_IRQ
- net BMV080_IRQ: now also J2.12 (IRQ)
- net ~{RESET_NPM1300} renamed ~{ENS160_INT}
- net ~{ENS160_INT}: now also U6.6 (~{INT})
- new net: J3.B5 (CC2), R3.2
- new net: J3.A5 (CC1), R4.1
- new net 5V: C28.1, C29.1, L2.2, U7.1 (IN)
- new net SHT41_SCL: IC1.8 (SCL_C), U3.2 (SCL)
- new net SHT41_SDA: IC1.2 (SDA_C), U3.1 (SDA)
- new net VUSB: C27.1, J3.A4_B9 (VBUS), J3.B4_A9 (VBUS__1), L2.1
- new net ~{ENS160_CS}: U1.12 (GPIO8), U6.7 (~{CS})
- no-connect marks 13 -> 25
Other:
- moved on the sheet: C20, C22, D2, R28, R9, U2, Um1
